File: um66t.brd (EAGLE design)
At the start: 50 x 50 mm, 12 parts, among them IC1 7833, T1 BC547

Commit message: Replaced 7833 with 10E resistor
Changed BC547 Package
Parts:
- removed IC1: 7833, linear:TO220V
- added R3: 100E, resistor:0204/5
- T1: value BC547 -> (none); device transistor:TO92 -> transistor:TO92-CBE
- moved LOGO1 49.0 mm to (22.0, 58.0)
- moved T1 1.00 mm to (58.2, 63.1)
Connections:
- net 5V: now also R3.2; no longer IC1.3
- net GND: now also T1.E; no longer IC1.2, T1.1
- net N$2: now also R3.1; no longer IC1.1
- net N$6: now also T1.B; no longer T1.2
- net N$7: now also T1.C; no longer T1.3
Routing:
- net GND: track 99.4 -> 90.4 mm
- net 5V: track 33.5 -> 29.3 mm
- net N$2: track 42.2 -> 45.2 mm
- net N$6: track 8.19 -> 9.21 mm
Changed lines of the file:
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@@
 <attribute name="VALUE" x="36.21" y="52.05" size="1.27" layer="27" ratio="10" rot="R270"/>
-</element>
-<element name="IC1" library="linear" library_urn="urn:adsk.eagle:library:262" package="TO220V" package3d_urn="urn:adsk.eagle:package:16417/2" value="7833" x="27.52" y="59.89" smashed="yes">
-<attribute name="NAME" x="22.44" y="53.8448" size="1.27" layer="25" ratio="10"/>
-<attribute name="VALUE" x="22.44" y="52.27" size="1.27" layer="27" ratio="10"/>
 </element>
 <element name="JP1" library="pinhead" library_urn="urn:adsk.eagle:library:325" package="1X02" package3d_urn="urn:adsk.eagle:package:22435/2" value="9V Battery" x="24.51" y="30.32" smashed="yes" rot="R270">
@@
 <attribute name="VALUE" x="19.27" y="50.13" size="1.778" layer="27" rot="R270"/>
 </element>
-<element name="T1" library="transistor" library_urn="urn:adsk.eagle:library:402" package="TO92" package3d_urn="urn:adsk.eagle:package:28523/2" value="BC547" x="59.17" y="63.14" smashed="yes" rot="R90">
-<attribute name="NAME" x="62.685" y="66.535" size="1.27" layer="25" ratio="10" rot="R180"/>
-<attribute name="VALUE" x="56.685" y="65.44" size="1.27" layer="27" ratio="10" rot="R180"/>
+<element name="T1" library="transistor" library_urn="urn:adsk.eagle:library:402" package="TO92-CBE" package3d_urn="urn:adsk.eagle:package:29921/2" value="" x="58.17" y="63.14" smashed="yes" rot="R90">
+<attribute name="NAME" x="61.685" y="66.535" size="1.27" layer="25" ratio="10" rot="R180"/>
+<attribute name="VALUE" x="55.685" y="65.44" size="1.27" layer="27" ratio="10" rot="R180"/>
 </element>
 <element name="R2" library="resistor" library_urn="urn:adsk.eagle:library:348" package="0204/5" package3d_urn="urn:adsk.eagle:package:23488/1" value="220E" x="27" y="25" smashed="yes" rot="R180">
@@
 <attribute name="VALUE" x="39.2004" y="23.1966" size="1.27" layer="27" ratio="10"/>
 </element>
-<element name="LOGO1" library="SparkFun-Aesthetics" library_urn="urn:adsk.eagle:library:507" package="OSHW-LOGO-M_COPPER" value="OSHW-LOGOM-COPPER" x="21" y="9" smashed="yes"/>
+<element name="LOGO1" library="SparkFun-Aesthetics" library_urn="urn:adsk.eagle:library:507" package="OSHW-LOGO-M_COPPER" value="OSHW-LOGOM-COPPER" x="22" y="58" smashed="yes"/>
+<element name="R3" library="resistor" library_urn="urn:adsk.eagle:library:348" package="0204/5" package3d_urn="urn:adsk.eagle:package:23488/1" value="100E" x="32" y="57" smashed="yes">
+<attribute name="NAME" x="29.9934" y="58.1684" size="0.9906" layer="25" ratio="10"/>
+<attribute name="VALUE" x="29.8664" y="54.6886" size="0.9906" layer="27" ratio="10"/>
+</element>
 </elements>
 <signals>
@@
 <signal name="N$2">
 <contactref element="S1" pad="1"/>
-<contactref element="IC1" pad="1"/>
-<wire x1="20" y1="50" x2="25" y2="55" width="1.27" layer="16"/>
-<wire x1="25" y1="55" x2="25" y2="57.33" width="1.27" layer="16"/>
-<wire x1="25" y1="57.33" x2="24.98" y2="57.35" width="1.27" layer="16"/>
 <contactref element="R2" pad="2"/>
 <wire x1="24.46" y1="25" x2="22" y2="25" width="1.27" layer="16"/>
@@
 <wire x1="24.35" y1="47.59" x2="20.41" y2="47.59" width="1.27" layer="16"/>
 <wire x1="20.41" y1="47.59" x2="20" y2="48" width="1.27" layer="16"/>
+<contactref element="R3" pad="1"/>
+<wire x1="27" y1="57" x2="29.46" y2="57" width="1.27" layer="16"/>
+<wire x1="20" y1="50" x2="27" y2="57" width="1.27" layer="16"/>
 </signal>
 <signal name="5V">
-<contactref element="IC1" pad="3"/>
 <contactref element="C2" pad="+"/>
 <contactref element="C1" pad="1"/>
 <contactref element="JP3" pad="2"/>
 <contactref element="JP2" pad="1"/>
-<wire x1="30.06" y1="57.35" x2="38.53" y2="57.35" width="1.27" layer="16"/>
 <wire x1="38.53" y1="57.35" x2="38.75" y2="57.13" width="1.27" layer="16"/>
 <wire x1="38.75" y1="57.13" x2="43.67" y2="57.13" width="1.27" layer="16"/>
@@
 <wire x1="54.55" y1="55" x2="59" y2="55" width="1.27" layer="16"/>
 <wire x1="59" y1="55" x2="60.05" y2="53.95" width="1.27" layer="16"/>
+<contactref element="R3" pad="2"/>
+<wire x1="38.75" y1="57.13" x2="34.67" y2="57.13" width="1.27" layer="16"/>
+<wire x1="34.67" y1="57.13" x2="34.54" y2="57" width="1.27" layer="16"/>
 </signal>
 <signal name="N$5">
@@
 </signal>
 <signal name="N$6">
-<contactref element="T1" pad="2"/>
+<contactref element="T1" pad="B"/>
 <contactref element="R1" pad="2"/>
-<wire x1="49.33" y1="63.75" x2="56.655" y2="63.75" width="1.27" layer="16"/>
-<wire x1="56.655" y1="63.75" x2="57.265" y2="63.14" width="1.27" layer="16"/>
+<wire x1="49.33" y1="63.75" x2="52.25" y2="63.75" width="1.27" layer="16"/>
+<wire x1="52.25" y1="63.75" x2="53" y2="63" width="1.27" layer="16"/>
+<wire x1="53" y1="63" x2="58.03" y2="63" width="1.27" layer="16"/>
+<wire x1="58.03" y1="63" x2="58.17" y2="63.14" width="1.27" layer="16"/>
 </signal>
 <signal name="N$7">
 <contactref element="JP2" pad="2"/>
-<contactref element="T1" pad="3"/>
-<wire x1="59.17" y1="61.87" x2="59.17" y2="57.83" width="1.27" layer="16"/>
-<wire x1="60.51" y1="56.49" x2="61.87" y2="56.49" width="1.27" layer="16"/>
-<wire x1="59.17" y1="57.83" x2="60.51" y2="56.49" width="1.27" layer="16"/>
+<contactref element="T1" pad="C"/>
+<wire x1="58.17" y1="60.6" x2="60.4" y2="60.6" width="1.27" layer="16"/>
+<wire x1="61.87" y1="59.13" x2="61.87" y2="56.49" width="1.27" layer="16"/>
+<wire x1="60.4" y1="60.6" x2="61.87" y2="59.13" width="1.27" layer="16"/>
 </signal>
 <signal name="GND">
 <contactref element="JP3" pad="1"/>
 <contactref element="JP1" pad="2"/>
-<contactref element="IC1" pad="2"/>
 <contactref element="C2" pad="-"/>
 <contactref element="C1" pad="2"/>
-<contactref element="T1" pad="1"/>
-<wire x1="27.52" y1="57.35" x2="27.52" y2="52.48" width="1.27" layer="16"/>
-<wire x1="27.52" y1="52.48" x2="28" y2="52" width="1.27" layer="16"/>
-<wire x1="28" y1="52" x2="33" y2="52" width="1.27" layer="16"/>
+<contactref element="T1" pad="E"/>
 <wire x1="33" y1="52" x2="38.7" y2="52" width="1.27" layer="16"/>
 <wire x1="38.7" y1="52" x2="38.75" y2="52.05" width="1.27" layer="16"/>
@@
 <wire x1="48" y1="52" x2="46.1" y2="52" width="1.27" layer="16"/>
 <wire x1="46.1" y1="52" x2="46.05" y2="52.05" width="1.27" layer="16"/>
-<wire x1="59.17" y1="64.41" x2="60.59" y2="64.41" width="1.27" layer="16"/>
-<wire x1="60.59" y1="64.41" x2="66" y2="59" width="1.27" layer="16"/>
-<wire x1="66" y1="59" x2="66" y2="53" width="1.27" layer="16"/>
-<wire x1="66" y1="53" x2="64" y2="51" width="1.27" layer="16"/>
+<wire x1="64" y1="51" x2="66" y2="53" width="1.27" layer="16"/>
 <wire x1="64" y1="51" x2="58" y2="51" width="1.27" layer="16"/>
 <wire x1="58" y1="51" x2="56.48" y2="52.52" width="1.27" layer="16"/>
@@
 <wire x1="37" y1="28" x2="35.95" y2="29.05" width="1.27" layer="16"/>
 <wire x1="33" y1="52" x2="33" y2="29.05" width="1.27" layer="16"/>
+<wire x1="66" y1="53" x2="66" y2="59" width="1.27" layer="16"/>
+<wire x1="66" y1="59" x2="59.32" y2="65.68" width="1.27" layer="16"/>
+<wire x1="59.32" y1="65.68" x2="58.17" y2="65.68" width="1.27" layer="16"/>
 </signal>
 <signal name="N$1">

Commit message: Changed 9V Battery to 5V Supply
Parts:
- JP1: value 9V Battery -> 5V Supply
- T1: value (none) -> BC547
Changed lines of the file:
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@@
 <attribute name="VALUE" x="36.21" y="52.05" size="1.27" layer="27" ratio="10" rot="R270"/>
 </element>
-<element name="JP1" library="pinhead" library_urn="urn:adsk.eagle:library:325" package="1X02" package3d_urn="urn:adsk.eagle:package:22435/2" value="9V Battery" x="24.51" y="30.32" smashed="yes" rot="R270">
+<element name="JP1" library="pinhead" library_urn="urn:adsk.eagle:library:325" package="1X02" package3d_urn="urn:adsk.eagle:package:22435/2" value="5V Supply" x="24.51" y="30.32" smashed="yes" rot="R270">
 <attribute name="NAME" x="26.3388" y="32.9362" size="1.27" layer="25" ratio="10" rot="R270"/>
-<attribute name="VALUE" x="21.335" y="32.86" size="1.27" layer="27" rot="R270"/>
+<attribute name="VALUE" x="21.335" y="34.86" size="1.27" layer="27" rot="R270"/>
 </element>
 <element name="JP2" library="pinhead" library_urn="urn:adsk.eagle:library:325" package="1X02" package3d_urn="urn:adsk.eagle:package:22435/2" value="Speaker" x="61.87" y="55.22" smashed="yes" rot="R90">
@@
 <attribute name="VALUE" x="19.27" y="50.13" size="1.778" layer="27" rot="R270"/>
 </element>
-<element name="T1" library="transistor" library_urn="urn:adsk.eagle:library:402" package="TO92-CBE" package3d_urn="urn:adsk.eagle:package:29921/2" value="" x="58.17" y="63.14" smashed="yes" rot="R90">
+<element name="T1" library="transistor" library_urn="urn:adsk.eagle:library:402" package="TO92-CBE" package3d_urn="urn:adsk.eagle:package:29921/2" value="BC547" x="58.17" y="63.14" smashed="yes" rot="R90">
 <attribute name="NAME" x="61.685" y="66.535" size="1.27" layer="25" ratio="10" rot="R180"/>
-<attribute name="VALUE" x="55.685" y="65.44" size="1.27" layer="27" ratio="10" rot="R180"/>
+<attribute name="VALUE" x="55.44" y="60.315" size="1.27" layer="27" ratio="10" rot="R90"/>
 </element>
 <element name="R2" library="resistor" library_urn="urn:adsk.eagle:library:348" package="0204/5" package3d_urn="urn:adsk.eagle:package:23488/1" value="220E" x="27" y="25" smashed="yes" rot="R180">
